Commit message: Simulation draft

File: balltze_description/urdf/balltze_macro.urdf.xacro (robot description, xacro)
@@ -15,8 +15,8 @@
     <xacro:body.body />
     <!-- LED DECLARATION -->
-    <xacro:leg.leg leg_prefix="front_left"  robot_width="0.1" robot_length="0.2" />
-    <xacro:leg.leg leg_prefix="front_right" robot_width="0.1" robot_length="0.2" />
-    <xacro:leg.leg leg_prefix="rear_left"   robot_width="0.1" robot_length="0.2" />
-    <xacro:leg.leg leg_prefix="rear_right"  robot_width="0.1" robot_length="0.2" />
+    <xacro:leg.leg leg_prefix="front_left"  robot_width="0.15" robot_length="0.3" />
+    <xacro:leg.leg leg_prefix="front_right" robot_width="0.15" robot_length="0.3" />
+    <xacro:leg.leg leg_prefix="rear_left"   robot_width="0.15" robot_length="0.3" />
+    <xacro:leg.leg leg_prefix="rear_right"  robot_width="0.15" robot_length="0.3" />
     <xacro:control.ros2_control_system />
   </xacro:macro>

File: balltze_description/urdf/body.urdf.xacro (robot description, xacro)
@@ -6,5 +6,5 @@
       <visual>
         <geometry>
-          <mesh filename="$(find balltze_description)/meshes/body_link.stl" scale="1.0 1.0 1.0" />
+          <mesh filename="file://$(find balltze_description)/meshes/body_link.stl" scale="0.5 0.5 0.5" />
         </geometry>
         <origin xyz="0.0 0.0 0.0" rpy="0.0 0.0 0.0" />
@@ -12,5 +12,5 @@
       <collision>
         <geometry>
-          <mesh filename="$(find balltze_description)/meshes/body_link_colision.stl" scale="1.0 1.0 1.0" />
+          <mesh filename="file://$(find balltze_description)/meshes/body_link_collision.stl" scale="0.5 0.5 0.5" />
         </geometry>
         <origin xyz="0.0 0.0 0.0" rpy="0.0 0.0 0.0" />

File: balltze_description/urdf/gazebo.ros2_control.xacro (robot description, xacro)
@@ -3,16 +3,19 @@
     <xacro:macro name="ros2_control_system">
       <xacro:macro name="ros2_control_joint" params="joint_name">
+        <xacro:property name="motor_range"   value="${300.0 / 360.0 * (2.0 * pi)}" />
+        <xacro:property name="motor_max_vel" value="${114.0 * (2.0 * pi / 60.0)}" />
+        <xacro:property name="motor_max_eff" value="1.5" />
         <joint name="${joint_name}">
           <command_interface name="position">
-            <param name="min">-5.23</param>
-            <param name="max">5.23</param>
+            <param name="min">-${motor_range/2.0}</param>
+            <param name="max">${motor_range/2.0}</param>
           </command_interface>
           <command_interface name="velocity">
-            <param name="min">-11.932</param>
-            <param name="max">11.932</param>
+            <param name="min">-${motor_max_vel}</param>
+            <param name="max">${motor_max_vel}</param>
           </command_interface>
           <command_interface name="effort">
-            <param name="min">-1.50</param>
-            <param name="max">1.50</param>
+            <param name="min">-${motor_max_eff}</param>
+            <param name="max">${motor_max_eff}</param>
           </command_interface>
           <state_interface name="position">
@@ -39,6 +42,4 @@
       <gazebo>
         <plugin filename="libign_ros2_control-system.so" name="ign_ros2_control::IgnitionROS2ControlPlugin">
-          <robot_param>robot_description</robot_param>
-          <robot_param_node>robot_state_publisher</robot_param_node>
           <parameters>$(find balltze_description)/config/controllers.yaml</parameters>
         </plugin>

File: balltze_description/urdf/hardware.ros2_control.xacro (robot description, xacro)
@@ -10,5 +10,5 @@
           <state_interface name="velocity" />
           <state_interface name="effort" />
-          <id>${motor_id}</id>
+          <param name="id">${motor_id}</param>
         </joint>
       </xacro:macro>
@@ -20,9 +20,9 @@
       <ros2_control name="DynamixelSystem" type="system">
         <hardware>
-          <plugin>dynamixel_hardware_system/DynamixelAX12ASystem</plugin>
+          <plugin>balltze_dynamixel_system/BalltzeDynamixelSystem</plugin>
         </hardware>
-        <serial_port>/dev/ttyUSB1</serial_port>
-        <baudrate>1000000</baudrate>
-        <return_delay>50</return_delay>
+        <param name="serial_port">/dev/ttyUSB1</param>
+        <param name="baudrate">1000000</param>
+        <param name="return_delay">50</param>
         <xacro:leg_joints leg_prefix="front_left"  coxa_motor_id="0" />
         <xacro:leg_joints leg_prefix="front_right" coxa_motor_id="3" />

File: balltze_description/urdf/leg.urdf.xacro (robot description, xacro)
@@ -3,6 +3,7 @@
   <!-- LEG MACRO -->
   <xacro:macro name="leg" params="leg_prefix robot_width robot_length">
-    <xacro:property name="coxa_to_femur_x" value="0.1" />
-    <xacro:property name="coxa_to_femur_y" value="0.1" />
+    <xacro:property name="coxa_to_femur_x" value="0.0" />
+    <xacro:property name="coxa_to_femur_y" value="0.06" />
+    <xacro:property name="coxa_to_femur_z" value="0.0" />
     <xacro:macro name="coxa_inertial">
       <inertial>
@@ -11,7 +12,7 @@
       </inertial>
     </xacro:macro>
-    <xacro:property name="femur_to_tibia_x" value="0.1" />
-    <xacro:property name="femur_to_tibia_y" value="0.1" />
-    <xacro:property name="femur_to_tibia_z" value="0.1" />
+    <xacro:property name="femur_to_tibia_x" value="0.0" />
+    <xacro:property name="femur_to_tibia_y" value="0.0" />
+    <xacro:property name="femur_to_tibia_z" value="-0.11" />
     <xacro:macro name="femur_inertial">
       <inertial>
@@ -20,7 +21,7 @@
       </inertial>
     </xacro:macro>
-    <xacro:property name="tibia_to_tip_x" value="0.1" />
-    <xacro:property name="tibia_to_tip_y" value="0.1" />
-    <xacro:property name="tibia_to_tip_z" value="0.1" />
+    <xacro:property name="tibia_to_tip_x" value="0.15" />
+    <xacro:property name="tibia_to_tip_y" value="0.0" />
+    <xacro:property name="tibia_to_tip_z" value="0.0" />
     <xacro:macro name="tibia_inertial">
       <inertial>
@@ -29,9 +30,12 @@
       </inertial>
     </xacro:macro>
+    <xacro:property name="motor_range"   value="${300.0 / 360.0 * (2.0 * pi)}" />
+    <xacro:property name="motor_max_vel" value="${114.0 * (2.0 * pi / 60.0)}" />
+    <xacro:property name="motor_max_eff" value="1.5" />
     <!-- CONDITIONAL BLOCKS -->
     <xacro:if value="${leg_prefix == 'front_left'}">
       <xacro:property name="side" value="left" />
       <xacro:property name="body_to_coxa_xyz" value="${robot_length/2.0} ${robot_width/2.0} 0.0" />
-      <xacro:property name="coxa_to_femur_xyz" value="${coxa_to_femur_x} ${coxa_to_femur_y} 0.0" />
+      <xacro:property name="coxa_to_femur_xyz" value="${coxa_to_femur_x} ${coxa_to_femur_y} ${coxa_to_femur_z}" />
       <xacro:property name="femur_tibia_xyz" value="${femur_to_tibia_x} ${femur_to_tibia_y} ${femur_to_tibia_z}" />
       <xacro:property name="tibia_tip_xyz" value="${tibia_to_tip_x} ${tibia_to_tip_y} ${tibia_to_tip_z}" />
@@ -39,12 +43,12 @@
     <xacro:if value="${leg_prefix == 'front_right'}">
       <xacro:property name="side" value="left" />
-      <xacro:property name="body_to_coxa_xyz" value="${robot_length/2.0} ${robot_width/2.0} 0.0" />
-      <xacro:property name="coxa_to_femur_xyz" value="${coxa_to_femur_x} ${coxa_to_femur_y} 0.0" />
-      <xacro:property name="femur_tibia_xyz" value="${femur_to_tibia_x} ${femur_to_tibia_y} ${femur_to_tibia_z}" />
-      <xacro:property name="tibia_tip_xyz" value="${tibia_to_tip_x} ${tibia_to_tip_y} ${tibia_to_tip_z}" />
+      <xacro:property name="body_to_coxa_xyz" value="${robot_length/2.0} -${robot_width/2.0} 0.0" />
+      <xacro:property name="coxa_to_femur_xyz" value="${coxa_to_femur_x} -${coxa_to_femur_y} 0.0" />
+      <xacro:property name="femur_tibia_xyz" value="${femur_to_tibia_x} -${femur_to_tibia_y} ${femur_to_tibia_z}" />
+      <xacro:property name="tibia_tip_xyz" value="${tibia_to_tip_x} -${tibia_to_tip_y} ${tibia_to_tip_z}" />
     </xacro:if>
     <xacro:if value="${leg_prefix == 'rear_left'}">
       <xacro:property name="side" value="left" />
-      <xacro:property name="body_to_coxa_xyz" value="${robot_length/2.0} ${robot_width/2.0} 0.0" />
+      <xacro:property name="body_to_coxa_xyz" value="-${robot_length/2.0} ${robot_width/2.0} 0.0" />
       <xacro:property name="coxa_to_femur_xyz" value="${coxa_to_femur_x} ${coxa_to_femur_y} 0.0" />
       <xacro:property name="femur_tibia_xyz" value="${femur_to_tibia_x} ${femur_to_tibia_y} ${femur_to_tibia_z}" />
@@ -53,8 +57,8 @@
     <xacro:if value="${leg_prefix == 'rear_right'}">
       <xacro:property name="side" value="left" />
-      <xacro:property name="body_to_coxa_xyz" value="${robot_length/2.0} ${robot_width/2.0} 0.0" />
-      <xacro:property name="coxa_to_femur_xyz" value="${coxa_to_femur_x} ${coxa_to_femur_y} 0.0" />
-      <xacro:property name="femur_tibia_xyz" value="${femur_to_tibia_x} ${femur_to_tibia_y} ${femur_to_tibia_z}" />
-      <xacro:property name="tibia_tip_xyz" value="${tibia_to_tip_x} ${tibia_to_tip_y} ${tibia_to_tip_z}" />
+      <xacro:property name="body_to_coxa_xyz" value="-${robot_length/2.0} -${robot_width/2.0} 0.0" />
+      <xacro:property name="coxa_to_femur_xyz" value="${coxa_to_femur_x} -${coxa_to_femur_y} 0.0" />
+      <xacro:property name="femur_tibia_xyz" value="${femur_to_tibia_x} -${femur_to_tibia_y} ${femur_to_tibia_z}" />
+      <xacro:property name="tibia_tip_xyz" value="${tibia_to_tip_x} -${tibia_to_tip_y} ${tibia_to_tip_z}" />
     </xacro:if>
     <!-- LEG LINK -->
@@ -64,5 +68,5 @@
         <visual>
           <geometry>
-            <mesh filename="$(find balltze_description)/meshes/${side}_${link_name}.stl" scale="1.0 1.0 1.0" />
+            <mesh filename="file://$(find balltze_description)/meshes/${side}_${link_name}.stl" scale="0.1 0.1 0.1" />
           </geometry>
           <origin xyz="0.0 0.0 0.0" rpy="0.0 0.0 0.0" />
@@ -70,5 +74,5 @@
         <collision>
           <geometry>
-            <mesh filename="$(find balltze_description)/meshes/${side}_${link_name}_colision.stl" scale="1.0 1.0 1.0" />
+            <mesh filename="file://$(find balltze_description)/meshes/${side}_${link_name}_collision.stl" scale="0.1 0.1 0.1" />
           </geometry>
           <origin xyz="0.0 0.0 0.0" rpy="0.0 0.0 0.0" />
@@ -89,8 +93,11 @@
           <parent link="${leg_prefix}_${parent}" />
         </xacro:unless>
-        <child link="${leg_prefix}_${parent}" />
+        <child link="${leg_prefix}_${child}" />
         <origin xyz="${xyz}" rpy="0.0 0.0 0.0" />
         <axis xyz="${axis}" />
-        <limit effort="1.5" />
+        <limit effort="${motor_max_eff}"
+               lower="${motor_range/2.0}"
+               upper="${-motor_range/2.0}"
+               velocity="${motor_max_vel}" />
       </joint>
     </xacro:macro>
@@ -105,5 +112,18 @@
       <xacro:tibia_inertial/>
     </xacro:leg_link>
-    <link name="${leg_prefix}_tip_link"></link>
+    <link name="${leg_prefix}_tip_link">
+      <visual>
+        <geometry>
+          <mesh filename="file://$(find balltze_description)/meshes/${side}_coxa_link.stl" scale="0.1 0.1 0.1" />
+        </geometry>
+        <origin xyz="0.0 0.0 0.0" rpy="0.0 0.0 0.0" />
+      </visual>
+      <collision>
+        <geometry>
+          <mesh filename="file://$(find balltze_description)/meshes/${side}_coxa_link_collision.stl" scale="0.1 0.1 0.1" />
+        </geometry>
+        <origin xyz="0.0 0.0 0.0" rpy="0.0 0.0 0.0" />
+      </collision>
+    </link>
     <!-- DEFINE JOINTS -->
     <xacro:leg_joint

Commit message: Hardware working

File: balltze_description/urdf/balltze_macro.urdf.xacro (robot description, xacro)
@@ -14,4 +14,10 @@
     <!-- BODY DECLARATION -->
     <xacro:body.body />
+    <link name="world"></link>
+    <joint name="asdf" type="fixed">
+      <origin xyz="0.0 0.0 1.0" rpy="0.0 0.0 0.0"/>
+      <parent link="world"/>
+      <child link="base_link"/>
+    </joint>
     <!-- LED DECLARATION -->
     <xacro:leg.leg leg_prefix="front_left"  robot_width="0.15" robot_length="0.3" />

File: balltze_description/urdf/gazebo.ros2_control.xacro (robot description, xacro)
@@ -15,8 +15,8 @@
             <param name="max">${motor_max_vel}</param>
           </command_interface>
-          <command_interface name="effort">
+          <!-- <command_interface name="effort">
             <param name="min">-${motor_max_eff}</param>
             <param name="max">${motor_max_eff}</param>
-          </command_interface>
+          </command_interface> -->
           <state_interface name="position">
             <param name="initial_value">${init_pos}</param>

File: balltze_description/urdf/hardware.ros2_control.xacro (robot description, xacro)
@@ -25,8 +25,8 @@
           <param name="return_delay">50</param>
         </hardware>
-        <xacro:leg_joints leg_prefix="front_left"  coxa_motor_id="10" />
-        <!-- <xacro:leg_joints leg_prefix="front_right" coxa_motor_id="3" />
-        <xacro:leg_joints leg_prefix="rear_left"   coxa_motor_id="6" />
-        <xacro:leg_joints leg_prefix="rear_right"  coxa_motor_id="9" /> -->
+        <xacro:leg_joints leg_prefix="front_left"  coxa_motor_id="1" />
+        <xacro:leg_joints leg_prefix="front_right" coxa_motor_id="4" />
+        <!-- <xacro:leg_joints leg_prefix="rear_left"   coxa_motor_id="7" /> -->
+        <!-- <xacro:leg_joints leg_prefix="rear_right"  coxa_motor_id="10" /> -->
       </ros2_control>
     </xacro:macro>

File: balltze_description/urdf/leg.urdf.xacro (robot description, xacro)
@@ -9,5 +9,5 @@
       <inertial>
         <mass value="0.1" />
-        <inertia ixx="1" ixy="0" ixz="0" iyy="1" iyz="0" izz="1" />
+        <inertia ixx="0.01" ixy="0" ixz="0" iyy="0.01" iyz="0" izz="0.01" />
       </inertial>
     </xacro:macro>
@@ -18,5 +18,5 @@
       <inertial>
         <mass value="0.1" />
-        <inertia ixx="1" ixy="0" ixz="0" iyy="1" iyz="0" izz="1" />
+        <inertia ixx="0.01" ixy="0" ixz="0" iyy="0.01" iyz="0" izz="0.01" />
       </inertial>
     </xacro:macro>
@@ -27,5 +27,5 @@
       <inertial>
         <mass value="0.1" />
-        <inertia ixx="1" ixy="0" ixz="0" iyy="1" iyz="0" izz="1" />
+        <inertia ixx="0.01" ixy="0" ixz="0" iyy="0.01" iyz="0" izz="0.01" />
       </inertial>
     </xacro:macro>
@@ -84,5 +84,5 @@
     </xacro:macro>
     <!-- LEG JOINT -->
-    <xacro:macro name="leg_joint" params="leg_prefix parent child xyz axis">
+    <xacro:macro name="leg_joint" params="leg_prefix parent child xyz axis joint_min joint_max">
       <!-- JOINT DEFINITION -->
       <joint name="${leg_prefix}_${parent}_to_${child}_joint" type="revolute">
@@ -96,8 +96,8 @@
         <origin xyz="${xyz}" rpy="0.0 0.0 0.0" />
         <axis xyz="${axis}" />
-        <dynamics damping="0.2"/>
+        <dynamics damping="0.0"/>
         <limit effort="${motor_max_eff}"
-               lower="${-motor_range/2.0}"
-               upper="${motor_range/2.0}"
+               lower="${joint_min}"
+               upper="${joint_max}"
                velocity="${motor_max_vel}" />
       </joint>
@@ -134,4 +134,6 @@
       xyz="${body_to_coxa_xyz}"
       axis="1 0 0"
+      joint_min="${-pi/4.0}"
+      joint_max="${pi/4.0}"
     />
     <xacro:leg_joint
@@ -141,4 +143,6 @@
       xyz="${coxa_to_femur_xyz}"
       axis="0 1 0"
+      joint_min="${-pi/2.0}"
+      joint_max="${pi/2.0}"
     />
     <xacro:leg_joint
@@ -148,4 +152,6 @@
       xyz="${femur_tibia_xyz}"
       axis="0 1 0"
+      joint_min="${-pi/2.0}"
+      joint_max="${pi/2.0}"
     />
     <joint name="${leg_prefix}_tibia_link_to_tip_link_joint" type="fixed">

Commit message: Fix controller manager issue

File: balltze_description/urdf/balltze_macro.urdf.xacro (robot description, xacro)
@@ -14,10 +14,4 @@
     <!-- BODY DECLARATION -->
     <xacro:body.body />
-    <link name="world"></link>
-    <joint name="asdf" type="fixed">
-      <origin xyz="0.0 0.0 1.0" rpy="0.0 0.0 0.0"/>
-      <parent link="world"/>
-      <child link="base_link"/>
-    </joint>
     <!-- LED DECLARATION -->
     <xacro:leg.leg leg_prefix="front_left"  robot_width="0.15" robot_length="0.3" />

File: balltze_description/urdf/gazebo.ros2_control.xacro (robot description, xacro)
@@ -42,5 +42,5 @@
       <gazebo>
         <plugin filename="ign_ros2_control-system" name="ign_ros2_control::IgnitionROS2ControlPlugin">
-          <parameters>$(find balltze_description)/config/controllers.yaml</parameters>
+          <parameters>$(find balltze_bringup)/config/controllers.yaml</parameters>
         </plugin>
       </gazebo>

File: balltze_description/urdf/hardware.ros2_control.xacro (robot description, xacro)
@@ -6,5 +6,5 @@
           <command_interface name="position" />
           <command_interface name="velocity" />
-          <command_interface name="effort" />
+          <!-- <command_interface name="effort" /> -->
           <state_interface name="position" />
           <state_interface name="velocity" />
@@ -27,6 +27,6 @@
         <xacro:leg_joints leg_prefix="front_left"  coxa_motor_id="1" />
         <xacro:leg_joints leg_prefix="front_right" coxa_motor_id="4" />
-        <!-- <xacro:leg_joints leg_prefix="rear_left"   coxa_motor_id="7" /> -->
-        <!-- <xacro:leg_joints leg_prefix="rear_right"  coxa_motor_id="10" /> -->
+        <xacro:leg_joints leg_prefix="rear_left"   coxa_motor_id="7" />
+        <xacro:leg_joints leg_prefix="rear_right"  coxa_motor_id="10" />
       </ros2_control>
     </xacro:macro>
