Commit message: Change collisions to spheres

File: balltze_description/urdf/body.urdf.xacro (robot description, xacro)
@@ -17,5 +17,5 @@
       </collision>
       <inertial>
-          <mass value="1.2" />
+          <mass value="2.2" />
           <inertia ixx="1.0" ixy="0.0" ixz="0.0"
                              iyy="1.0" iyz="0.0"

File: balltze_description/urdf/gazebo.ros2_control.xacro (robot description, xacro)
@@ -28,5 +28,5 @@
       <xacro:macro name="leg_joints" params="leg_prefix">
         <xacro:ros2_control_joint joint_name="${leg_prefix}_body_link_to_coxa_link_joint"   init_pos="0.0"/>
-        <xacro:ros2_control_joint joint_name="${leg_prefix}_coxa_link_to_femur_link_joint"  init_pos="${-pi/4}"/>
+        <xacro:ros2_control_joint joint_name="${leg_prefix}_coxa_link_to_femur_link_joint"  init_pos="${pi/4.0}"/>
         <xacro:ros2_control_joint joint_name="${leg_prefix}_femur_link_to_tibia_link_joint" init_pos="0.0"/>
       </xacro:macro>

File: balltze_description/urdf/leg.urdf.xacro (robot description, xacro)
@@ -74,5 +74,6 @@
         <collision>
           <geometry>
-            <mesh filename="file://$(find balltze_description)/meshes/${side}_${link_name}_collision.stl" scale="0.1 0.1 0.1" />
+            <sphere radius="0.02"/>
+            <!-- <mesh filename="file://$(find balltze_description)/meshes/${side}_${link_name}_collision.stl" scale="0.1 0.1 0.1" /> -->
           </geometry>
           <origin xyz="0.0 0.0 0.0" rpy="0.0 0.0 0.0" />
@@ -122,5 +123,6 @@
       <collision>
         <geometry>
-          <mesh filename="file://$(find balltze_description)/meshes/${side}_coxa_link_collision.stl" scale="0.1 0.1 0.1" />
+          <sphere radius="0.02"/>
+          <!-- <mesh filename="file://$(find balltze_description)/meshes/${side}_coxa_link_collision.stl" scale="0.1 0.1 0.1" /> -->
         </geometry>
         <origin xyz="0.0 0.0 0.0" rpy="0.0 0.0 0.0" />
