Commit message: Add setup for dev containers

File: balltze_description/urdf/balltze.urdf (robot description, URDF)
Before this commit: robot balltze, 14 links, 13 joints
Links:
- link base_link: mass 1.0 -> 10.0; geometry collision box size=0.5 0.2 0.1; visual box size=0.5 0.2 0.1
- link fl_coxa: geometry collision sphere radius=0.015; visual box size=0.03 0.03 0.03
- link fl_femur: geometry collision sphere radius=0.015; visual box size=0.16 0.03 0.03
- link fl_tibia: geometry collision sphere radius=0.015; visual box size=0.16 0.03 0.03
- link fr_coxa: geometry collision sphere radius=0.015; visual box size=0.03 0.03 0.03
- link fr_femur: geometry collision sphere radius=0.015; visual box size=0.16 0.03 0.03
- link fr_tibia: geometry collision sphere radius=0.015; visual box size=0.16 0.03 0.03
- link rl_coxa: geometry collision sphere radius=0.015; visual box size=0.03 0.03 0.03
- link rl_femur: geometry collision sphere radius=0.015; visual box size=0.16 0.03 0.03
- link rl_tibia: geometry collision sphere radius=0.015; visual box size=0.16 0.03 0.03
- link rr_coxa: geometry collision sphere radius=0.015; visual box size=0.03 0.03 0.03
- link rr_femur: geometry collision sphere radius=0.015; visual box size=0.16 0.03 0.03
- link rr_tibia: geometry collision sphere radius=0.015; visual box size=0.16 0.03 0.03
Joints:
- joint fl_base_link_to_coxa_joint: limit lower=-0.785398163 upper=0.785398163 effort=1.5 velocity=0.003141593 -> lower=-0.785398163 upper=0.785398163 effort=200 velocity=5.0; origin xyz=0.1 0.05 0.0 rpy=0 0 0 -> xyz=0.25 0.13 0.0 rpy=0 0 0
- joint fl_coxa_to_femur_joint: limit lower=-2.35619449 upper=1.570796327 effort=1.5 velocity=0.003141593 -> lower=-2.35619449 upper=1.570796327 effort=200 velocity=5.0
- joint fl_femur_to_tibia_joint: limit lower=0.0 upper=3.141592654 effort=1.5 velocity=0.003141593 -> lower=0.0 upper=3.141592654 effort=200 velocity=5.0; origin xyz=0.06 0.0 0.0 rpy=0 0 0 -> xyz=0.16 0.0 0.0 rpy=0 0 0
- joint fr_base_link_to_coxa_joint: limit lower=-0.785398163 upper=0.785398163 effort=1.5 velocity=0.003141593 -> lower=-0.785398163 upper=0.785398163 effort=200 velocity=5.0; origin xyz=0.1 -0.05 0.0 rpy=0 0 0 -> xyz=0.25 -0.13 0.0 rpy=0 0 0
- joint fr_coxa_to_femur_joint: limit lower=-2.35619449 upper=1.570796327 effort=1.5 velocity=0.003141593 -> lower=-2.35619449 upper=1.570796327 effort=200 velocity=5.0
- joint fr_femur_to_tibia_joint: limit lower=0.0 upper=3.141592654 effort=1.5 velocity=0.003141593 -> lower=0.0 upper=3.141592654 effort=200 velocity=5.0; origin xyz=0.06 0.0 0.0 rpy=0 0 0 -> xyz=0.16 0.0 0.0 rpy=0 0 0
- joint rl_base_link_to_coxa_joint: limit lower=-0.785398163 upper=0.785398163 effort=1.5 velocity=0.003141593 -> lower=-0.785398163 upper=0.785398163 effort=200 velocity=5.0; origin xyz=-0.1 0.05 0.0 rpy=0 0 0 -> xyz=-0.25 0.13 0.0 rpy=0 0 0
- joint rl_coxa_to_femur_joint: limit lower=-2.35619449 upper=1.570796327 effort=1.5 velocity=0.003141593 -> lower=-2.35619449 upper=1.570796327 effort=200 velocity=5.0
- joint rl_femur_to_tibia_joint: limit lower=0.0 upper=3.141592654 effort=1.5 velocity=0.003141593 -> lower=0.0 upper=3.141592654 effort=200 velocity=5.0; origin xyz=0.06 0.0 0.0 rpy=0 0 0 -> xyz=0.16 0.0 0.0 rpy=0 0 0
- joint rr_base_link_to_coxa_joint: limit lower=-0.785398163 upper=0.785398163 effort=1.5 velocity=0.003141593 -> lower=-0.785398163 upper=0.785398163 effort=200 velocity=5.0; origin xyz=-0.1 -0.05 0.0 rpy=0 0 0 -> xyz=-0.25 -0.13 0.0 rpy=0 0 0
- joint rr_coxa_to_femur_joint: limit lower=-2.35619449 upper=1.570796327 effort=1.5 velocity=0.003141593 -> lower=-2.35619449 upper=1.570796327 effort=200 velocity=5.0
- joint rr_femur_to_tibia_joint: limit lower=0.0 upper=3.141592654 effort=1.5 velocity=0.003141593 -> lower=0.0 upper=3.141592654 effort=200 velocity=5.0; origin xyz=0.06 0.0 0.0 rpy=0 0 0 -> xyz=0.16 0.0 0.0 rpy=0 0 0

Commit message: ros2_control in ign-gazebo

File: balltze_description/urdf/balltze.urdf (robot description, URDF)
Before this commit: robot balltze, 19 links, 18 joints
Joints:
- removed joint front_left_body_link_to_body_link_joint
- removed joint front_left_coxa_link_to_coxa_link_joint
- removed joint front_left_femur_link_to_femur_link_joint
- removed joint front_right_body_link_to_body_link_joint
- removed joint front_right_coxa_link_to_coxa_link_joint
- removed joint front_right_femur_link_to_femur_link_joint
- removed joint rear_left_body_link_to_body_link_joint
- removed joint rear_left_coxa_link_to_coxa_link_joint
- removed joint rear_left_femur_link_to_femur_link_joint
- removed joint rear_right_body_link_to_body_link_joint
- removed joint rear_right_coxa_link_to_coxa_link_joint
- removed joint rear_right_femur_link_to_femur_link_joint
- added joint front_left_body_link_to_coxa_link_joint: type revolute, parent body_link, child front_left_coxa_link, origin xyz=0.15 0.075 0.0 rpy=0.0 0.0 0.0, axis 1 0 0, limit lower=-2.6179938779914944 upper=2.6179938779914944 effort=1.5 velocity=11.938052083641214
- added joint front_left_coxa_link_to_femur_link_joint: type revolute, parent front_left_coxa_link, child front_left_femur_link, origin xyz=0.0 0.06 0.0 rpy=0.0 0.0 0.0, axis 0 1 0, limit lower=-2.6179938779914944 upper=2.6179938779914944 effort=1.5 velocity=11.938052083641214
- added joint front_left_femur_link_to_tibia_link_joint: type revolute, parent front_left_femur_link, child front_left_tibia_link, origin xyz=0.0 0.0 -0.11 rpy=0.0 0.0 0.0, axis 0 1 0, limit lower=-2.6179938779914944 upper=2.6179938779914944 effort=1.5 velocity=11.938052083641214
- added joint front_right_body_link_to_coxa_link_joint: type revolute, parent body_link, child front_right_coxa_link, origin xyz=0.15 -0.075 0.0 rpy=0.0 0.0 0.0, axis 1 0 0, limit lower=-2.6179938779914944 upper=2.6179938779914944 effort=1.5 velocity=11.938052083641214
- added joint front_right_coxa_link_to_femur_link_joint: type revolute, parent front_right_coxa_link, child front_right_femur_link, origin xyz=0.0 -0.06 0.0 rpy=0.0 0.0 0.0, axis 0 1 0, limit lower=-2.6179938779914944 upper=2.6179938779914944 effort=1.5 velocity=11.938052083641214
- added joint front_right_femur_link_to_tibia_link_joint: type revolute, parent front_right_femur_link, child front_right_tibia_link, origin xyz=0.0 -0.0 -0.11 rpy=0.0 0.0 0.0, axis 0 1 0, limit lower=-2.6179938779914944 upper=2.6179938779914944 effort=1.5 velocity=11.938052083641214
- added joint rear_left_body_link_to_coxa_link_joint: type revolute, parent body_link, child rear_left_coxa_link, origin xyz=-0.15 0.075 0.0 rpy=0.0 0.0 0.0, axis 1 0 0, limit lower=-2.6179938779914944 upper=2.6179938779914944 effort=1.5 velocity=11.938052083641214
- added joint rear_left_coxa_link_to_femur_link_joint: type revolute, parent rear_left_coxa_link, child rear_left_femur_link, origin xyz=0.0 0.06 0.0 rpy=0.0 0.0 0.0, axis 0 1 0, limit lower=-2.6179938779914944 upper=2.6179938779914944 effort=1.5 velocity=11.938052083641214
- added joint rear_left_femur_link_to_tibia_link_joint: type revolute, parent rear_left_femur_link, child rear_left_tibia_link, origin xyz=0.0 0.0 -0.11 rpy=0.0 0.0 0.0, axis 0 1 0, limit lower=-2.6179938779914944 upper=2.6179938779914944 effort=1.5 velocity=11.938052083641214
- added joint rear_right_body_link_to_coxa_link_joint: type revolute, parent body_link, child rear_right_coxa_link, origin xyz=-0.15 -0.075 0.0 rpy=0.0 0.0 0.0, axis 1 0 0, limit lower=-2.6179938779914944 upper=2.6179938779914944 effort=1.5 velocity=11.938052083641214
- added joint rear_right_coxa_link_to_femur_link_joint: type revolute, parent rear_right_coxa_link, child rear_right_femur_link, origin xyz=0.0 -0.06 0.0 rpy=0.0 0.0 0.0, axis 0 1 0, limit lower=-2.6179938779914944 upper=2.6179938779914944 effort=1.5 velocity=11.938052083641214
- added joint rear_right_femur_link_to_tibia_link_joint: type revolute, parent rear_right_femur_link, child rear_right_tibia_link, origin xyz=0.0 -0.0 -0.11 rpy=0.0 0.0 0.0, axis 0 1 0, limit lower=-2.6179938779914944 upper=2.6179938779914944 effort=1.5 velocity=11.938052083641214
- joint base_link_to_body_link_joint: origin xyz=0.0 0.0 0.0 rpy=0.0 0.0 0.0 -> xyz=0.0 0.0 0.002 rpy=0.0 0.0 0.0
- joint body_link_to_imu_link_joint: origin xyz=0.0 0.0 0.0 rpy=0.0 0.0 0.0 -> xyz=0.0 0.0 0.01 rpy=0.0 0.0 0.0

File: balltze_description/urdf/body.urdf.xacro (robot description, xacro)
@@ -25,10 +25,10 @@
     <link name="imu_link"></link>
     <joint name="base_link_to_body_link_joint" type="fixed">
-      <origin xyz="0.0 0.0 0.0" rpy="0.0 0.0 0.0"/>
+      <origin xyz="0.0 0.0 0.002" rpy="0.0 0.0 0.0"/>
       <parent link="base_link"/>
       <child link="body_link"/>
     </joint>
     <joint name="body_link_to_imu_link_joint" type="fixed">
-      <origin xyz="0.0 0.0 0.0" rpy="0.0 0.0 0.0"/>
+      <origin xyz="0.0 0.0 0.01" rpy="0.0 0.0 0.0"/>
       <parent link="body_link"/>
       <child link="imu_link"/>

File: balltze_description/urdf/gazebo.ros2_control.xacro (robot description, xacro)
@@ -2,5 +2,5 @@
 <robot xmlns:xacro="http://wiki.ros.org/xacro">
     <xacro:macro name="ros2_control_system">
-      <xacro:macro name="ros2_control_joint" params="joint_name">
+      <xacro:macro name="ros2_control_joint" params="joint_name init_pos">
         <xacro:property name="motor_range"   value="${300.0 / 360.0 * (2.0 * pi)}" />
         <xacro:property name="motor_max_vel" value="${114.0 * (2.0 * pi / 60.0)}" />
@@ -20,5 +20,5 @@
           </command_interface>
           <state_interface name="position">
-            <param name="initial_value">0.0</param>
+            <param name="initial_value">${init_pos}</param>
           </state_interface>
           <state_interface name="velocity" />
@@ -27,7 +27,7 @@
       </xacro:macro>
       <xacro:macro name="leg_joints" params="leg_prefix">
-        <xacro:ros2_control_joint joint_name="${leg_prefix}_body_link_to_coxa_link_joint" />
-        <xacro:ros2_control_joint joint_name="${leg_prefix}_coxa_link_to_femur_link_joint" />
-        <xacro:ros2_control_joint joint_name="${leg_prefix}_femur_link_to_tibia_link_joint" />
+        <xacro:ros2_control_joint joint_name="${leg_prefix}_body_link_to_coxa_link_joint"   init_pos="0.0"/>
+        <xacro:ros2_control_joint joint_name="${leg_prefix}_coxa_link_to_femur_link_joint"  init_pos="${-pi/4}"/>
+        <xacro:ros2_control_joint joint_name="${leg_prefix}_femur_link_to_tibia_link_joint" init_pos="0.0"/>
       </xacro:macro>
       <ros2_control name="IgnitionSystem" type="system">
@@ -41,5 +41,5 @@
       </ros2_control>
       <gazebo>
-        <plugin filename="libign_ros2_control-system.so" name="ign_ros2_control::IgnitionROS2ControlPlugin">
+        <plugin filename="ign_ros2_control-system" name="ign_ros2_control::IgnitionROS2ControlPlugin">
           <parameters>$(find balltze_description)/config/controllers.yaml</parameters>
         </plugin>

File: balltze_description/urdf/leg.urdf.xacro (robot description, xacro)
@@ -8,5 +8,5 @@
     <xacro:macro name="coxa_inertial">
       <inertial>
-        <mass value="0.00000000001" />
+        <mass value="0.1" />
         <inertia ixx="1" ixy="0" ixz="0" iyy="1" iyz="0" izz="1" />
       </inertial>
@@ -17,5 +17,5 @@
     <xacro:macro name="femur_inertial">
       <inertial>
-        <mass value="0.00000000001" />
+        <mass value="0.1" />
         <inertia ixx="1" ixy="0" ixz="0" iyy="1" iyz="0" izz="1" />
       </inertial>
@@ -26,5 +26,5 @@
     <xacro:macro name="tibia_inertial">
       <inertial>
-        <mass value="0.00000000001" />
+        <mass value="0.1" />
         <inertia ixx="1" ixy="0" ixz="0" iyy="1" iyz="0" izz="1" />
       </inertial>
@@ -86,5 +86,5 @@
     <xacro:macro name="leg_joint" params="leg_prefix parent child xyz axis">
       <!-- JOINT DEFINITION -->
-      <joint name="${leg_prefix}_${parent}_to_${parent}_joint" type="revolute">
+      <joint name="${leg_prefix}_${parent}_to_${child}_joint" type="revolute">
         <xacro:if value="${parent == 'body_link'}">
           <parent link="${parent}" />
@@ -96,7 +96,8 @@
         <origin xyz="${xyz}" rpy="0.0 0.0 0.0" />
         <axis xyz="${axis}" />
+        <dynamics damping="0.2"/>
         <limit effort="${motor_max_eff}"
-               lower="${motor_range/2.0}"
-               upper="${-motor_range/2.0}"
+               lower="${-motor_range/2.0}"
+               upper="${motor_range/2.0}"
                velocity="${motor_max_vel}" />
       </joint>
