Commit message: Initial champ config

File: balltze_description/urdf/balltze.urdf (robot description, URDF)
Before this commit: robot balltze, 19 links, 18 joints
Links:
- removed link front_left_coxa_link
- removed link front_left_femur_link
- removed link front_left_tibia_link
- removed link front_left_tip_link
- removed link front_right_coxa_link
- removed link front_right_femur_link
- removed link front_right_tibia_link
- removed link front_right_tip_link
- removed link rear_left_coxa_link
- removed link rear_left_femur_link
- removed link rear_left_tibia_link
- removed link rear_left_tip_link
- removed link rear_right_coxa_link
- removed link rear_right_femur_link
- removed link rear_right_tibia_link
- removed link rear_right_tip_link
- added link fl_link_1, mass 0.1; collision sphere radius=0.02; visual sphere radius=0.02
- added link fl_link_2, mass 0.1; collision sphere radius=0.02; visual sphere radius=0.02
- added link fl_link_3, mass 0.1; collision sphere radius=0.02; visual sphere radius=0.02
- added link fl_tip; collision sphere radius=0.02; visual sphere radius=0.02
- added link fr_link_1, mass 0.1; collision sphere radius=0.02; visual sphere radius=0.02
- added link fr_link_2, mass 0.1; collision sphere radius=0.02; visual sphere radius=0.02
- added link fr_link_3, mass 0.1; collision sphere radius=0.02; visual sphere radius=0.02
- added link fr_tip; collision sphere radius=0.02; visual sphere radius=0.02
- added link rl_link_1, mass 0.1; collision sphere radius=0.02; visual sphere radius=0.02
- added link rl_link_2, mass 0.1; collision sphere radius=0.02; visual sphere radius=0.02
- added link rl_link_3, mass 0.1; collision sphere radius=0.02; visual sphere radius=0.02
- added link rl_tip; collision sphere radius=0.02; visual sphere radius=0.02
- added link rr_link_1, mass 0.1; collision sphere radius=0.02; visual sphere radius=0.02
- added link rr_link_2, mass 0.1; collision sphere radius=0.02; visual sphere radius=0.02
- added link rr_link_3, mass 0.1; collision sphere radius=0.02; visual sphere radius=0.02
- added link rr_tip; collision sphere radius=0.02; visual sphere radius=0.02
- link body_link: mass 1.2 -> 1.0
Joints:
- removed joint front_left_body_link_to_coxa_link_joint
- removed joint front_left_coxa_link_to_femur_link_joint
- removed joint front_left_femur_link_to_tibia_link_joint
- removed joint front_left_tibia_link_to_tip_link_joint
- removed joint front_right_body_link_to_coxa_link_joint
- removed joint front_right_coxa_link_to_femur_link_joint
- removed joint front_right_femur_link_to_tibia_link_joint
- removed joint front_right_tibia_link_to_tip_link_joint
- removed joint rear_left_body_link_to_coxa_link_joint
- removed joint rear_left_coxa_link_to_femur_link_joint
- removed joint rear_left_femur_link_to_tibia_link_joint
- removed joint rear_left_tibia_link_to_tip_link_joint
- removed joint rear_right_body_link_to_coxa_link_joint
- removed joint rear_right_coxa_link_to_femur_link_joint
- removed joint rear_right_femur_link_to_tibia_link_joint
- removed joint rear_right_tibia_link_to_tip_link_joint
- added joint fl_joint_1: type revolute, parent body_link, child fl_link_1, origin xyz=0.15 0.075 0.0 rpy=0.0 0.0 0.0, axis 1 0 0, limit lower=-0.7853981633974483 upper=0.7853981633974483 effort=1.5 velocity=11.938052083641214
- added joint fl_joint_2: type revolute, parent fl_link_1, child fl_link_2, origin xyz=0.0 0.06 0.0 rpy=0.0 0.0 0.0, axis 0 1 0, limit lower=-1.5707963267948966 upper=1.5707963267948966 effort=1.5 velocity=11.938052083641214
- added joint fl_joint_3: type revolute, parent fl_link_2, child fl_link_3, origin xyz=0.0 0.0 -0.11 rpy=0.0 0.0 0.0, axis 0 1 0, limit lower=-1.5707963267948966 upper=1.5707963267948966 effort=1.5 velocity=11.938052083641214
- added joint fl_joint_4: type fixed, parent fl_link_3, child fl_tip, origin xyz=0.15 0.0 0.0 rpy=0.0 0.0 0.0
- added joint fr_joint_1: type revolute, parent body_link, child fr_link_1, origin xyz=0.15 -0.075 0.0 rpy=0.0 0.0 0.0, axis 1 0 0, limit lower=-0.7853981633974483 upper=0.7853981633974483 effort=1.5 velocity=11.938052083641214
- added joint fr_joint_2: type revolute, parent fr_link_1, child fr_link_2, origin xyz=0.0 -0.06 0.0 rpy=0.0 0.0 0.0, axis 0 1 0, limit lower=-1.5707963267948966 upper=1.5707963267948966 effort=1.5 velocity=11.938052083641214
- added joint fr_joint_3: type revolute, parent fr_link_2, child fr_link_3, origin xyz=0.0 -0.0 -0.11 rpy=0.0 0.0 0.0, axis 0 1 0, limit lower=-1.5707963267948966 upper=1.5707963267948966 effort=1.5 velocity=11.938052083641214
- added joint fr_joint_4: type fixed, parent fr_link_3, child fr_tip, origin xyz=0.15 -0.0 0.0 rpy=0.0 0.0 0.0
- added joint rl_joint_1: type revolute, parent body_link, child rl_link_1, origin xyz=-0.15 0.075 0.0 rpy=0.0 0.0 0.0, axis 1 0 0, limit lower=-0.7853981633974483 upper=0.7853981633974483 effort=1.5 velocity=11.938052083641214
- added joint rl_joint_2: type revolute, parent rl_link_1, child rl_link_2, origin xyz=0.0 0.06 0.0 rpy=0.0 0.0 0.0, axis 0 1 0, limit lower=-1.5707963267948966 upper=1.5707963267948966 effort=1.5 velocity=11.938052083641214
- added joint rl_joint_3: type revolute, parent rl_link_2, child rl_link_3, origin xyz=0.0 0.0 -0.11 rpy=0.0 0.0 0.0, axis 0 1 0, limit lower=-1.5707963267948966 upper=1.5707963267948966 effort=1.5 velocity=11.938052083641214
- added joint rl_joint_4: type fixed, parent rl_link_3, child rl_tip, origin xyz=0.15 0.0 0.0 rpy=0.0 0.0 0.0
- added joint rr_joint_1: type revolute, parent body_link, child rr_link_1, origin xyz=-0.15 -0.075 0.0 rpy=0.0 0.0 0.0, axis 1 0 0, limit lower=-0.7853981633974483 upper=0.7853981633974483 effort=1.5 velocity=11.938052083641214
- added joint rr_joint_2: type revolute, parent rr_link_1, child rr_link_2, origin xyz=0.0 -0.06 0.0 rpy=0.0 0.0 0.0, axis 0 1 0, limit lower=-1.5707963267948966 upper=1.5707963267948966 effort=1.5 velocity=11.938052083641214
- added joint rr_joint_3: type revolute, parent rr_link_2, child rr_link_3, origin xyz=0.0 -0.0 -0.11 rpy=0.0 0.0 0.0, axis 0 1 0, limit lower=-1.5707963267948966 upper=1.5707963267948966 effort=1.5 velocity=11.938052083641214
- added joint rr_joint_4: type fixed, parent rr_link_3, child rr_tip, origin xyz=0.15 -0.0 0.0 rpy=0.0 0.0 0.0

File: balltze_description/urdf/balltze_macro.urdf.xacro (robot description, xacro)
@@ -15,8 +15,8 @@
     <xacro:body.body />
     <!-- LED DECLARATION -->
-    <xacro:leg.leg leg_prefix="front_left"  robot_width="0.15" robot_length="0.3" />
-    <xacro:leg.leg leg_prefix="front_right" robot_width="0.15" robot_length="0.3" />
-    <xacro:leg.leg leg_prefix="rear_left"   robot_width="0.15" robot_length="0.3" />
-    <xacro:leg.leg leg_prefix="rear_right"  robot_width="0.15" robot_length="0.3" />
+    <xacro:leg.leg leg_prefix="fl" robot_width="0.15" robot_length="0.3" />
+    <xacro:leg.leg leg_prefix="fr" robot_width="0.15" robot_length="0.3" />
+    <xacro:leg.leg leg_prefix="rl" robot_width="0.15" robot_length="0.3" />
+    <xacro:leg.leg leg_prefix="rr" robot_width="0.15" robot_length="0.3" />
     <xacro:control.ros2_control_system />
   </xacro:macro>

File: balltze_description/urdf/body.urdf.xacro (robot description, xacro)
@@ -17,8 +17,8 @@
       </collision>
       <inertial>
-          <mass value="2.2" />
-          <inertia ixx="1.0" ixy="0.0" ixz="0.0"
-                             iyy="1.0" iyz="0.0"
-                                       izz="1.0" />
+          <mass value="1.0" />
+          <inertia ixx="0.1" ixy="0.0" ixz="0.0"
+                             iyy="0.1" iyz="0.0"
+                                       izz="0.1" />
       </inertial>
     </link>
@@ -34,4 +34,12 @@
       <child link="imu_link"/>
     </joint>
+    <gazebo reference="imu_link">
+      <sensor name="imu_sensor" type="imu">
+        <always_on>1</always_on>
+        <update_rate>50.0</update_rate>
+        <visualize>true</visualize>
+        <topic>imu</topic>
+      </sensor>
+    </gazebo>
   </xacro:macro>
 </robot>

File: balltze_description/urdf/gazebo.ros2_control.xacro (robot description, xacro)
@@ -3,11 +3,11 @@
     <xacro:macro name="ros2_control_system">
       <xacro:macro name="ros2_control_joint" params="joint_name init_pos">
-        <xacro:property name="motor_range"   value="${300.0 / 360.0 * (2.0 * pi)}" />
+        <xacro:property name="motorrange"   value="${300.0 / 360.0 * (2.0 * pi)}" />
         <xacro:property name="motor_max_vel" value="${114.0 * (2.0 * pi / 60.0)}" />
         <xacro:property name="motor_max_eff" value="1.5" />
         <joint name="${joint_name}">
           <command_interface name="position">
-            <param name="min">-${motor_range/2.0}</param>
-            <param name="max">${motor_range/2.0}</param>
+            <param name="min">-${motorrange/2.0}</param>
+            <param name="max">${motorrange/2.0}</param>
           </command_interface>
           <command_interface name="velocity">
@@ -27,7 +27,7 @@
       </xacro:macro>
       <xacro:macro name="leg_joints" params="leg_prefix">
-        <xacro:ros2_control_joint joint_name="${leg_prefix}_body_link_to_coxa_link_joint"   init_pos="0.0"/>
-        <xacro:ros2_control_joint joint_name="${leg_prefix}_coxa_link_to_femur_link_joint"  init_pos="${pi/4.0}"/>
-        <xacro:ros2_control_joint joint_name="${leg_prefix}_femur_link_to_tibia_link_joint" init_pos="0.0"/>
+        <xacro:ros2_control_joint joint_name="${leg_prefix}_joint_1" init_pos="0.0"/>
+        <xacro:ros2_control_joint joint_name="${leg_prefix}_joint_2" init_pos="${pi/4.0}"/>
+        <xacro:ros2_control_joint joint_name="${leg_prefix}_joint_3" init_pos="0.0"/>
       </xacro:macro>
       <ros2_control name="IgnitionSystem" type="system">
@@ -35,12 +35,65 @@
           <plugin>ign_ros2_control/IgnitionSystem</plugin>
         </hardware>
-        <xacro:leg_joints leg_prefix="front_left" />
-        <xacro:leg_joints leg_prefix="front_right" />
-        <xacro:leg_joints leg_prefix="rear_left" />
-        <xacro:leg_joints leg_prefix="rear_right" />
+        <xacro:leg_joints leg_prefix="fl" />
+        <xacro:leg_joints leg_prefix="fr" />
+        <xacro:leg_joints leg_prefix="rl" />
+        <xacro:leg_joints leg_prefix="rr" />
+        <sensor name="imu_sensor">
+          <state_interface name="orientation.x"/>
+          <state_interface name="orientation.y"/>
+          <state_interface name="orientation.z"/>
+          <state_interface name="orientation.w"/>
+          <state_interface name="angular_velocity.x"/>
+          <state_interface name="angular_velocity.y"/>
+          <state_interface name="angular_velocity.z"/>
+          <state_interface name="linear_acceleration.x"/>
+          <state_interface name="linear_acceleration.y"/>
+          <state_interface name="linear_acceleration.z"/>
+        </sensor>
       </ros2_control>
+      <!-- <ros2_control name="BalltzeIgnitionTipSensor" type="system">
+        <hardware>
+          <plugin>balltze_simulation/TipSensor</plugin>
+        </hardware>
+        <gpio name="fl_tip">
+          <param name="topic">/balltze/fl_tip/contact</param>
+          <state_interface name="logical"/>
+            <param name="link">fl_tip</param>
+          <state_interface />
+        </gpio>
+        <gpio name="fr_tip">
+          <param name="topic">/balltze/fr_tip/contact</param>
+          <state_interface name="logical"/>
+            <param name="link">fr_tip</param>
+          <state_interface />
+        </gpio>
+        <gpio name="rl_tip">
+          <param name="topic">/balltze/rl_tip/contact</param>
+          <state_interface name="logical"/>
+            <param name="link">rl_tip</param>
+          <state_interface />
+        </gpio>
+        <gpio name="rr_tip">
+          <param name="topic">/balltze/rr_tip/contact</param>
+          <state_interface name="logical"/>
+            <param name="link">rr_tip</param>
+          <state_interface />
+        </gpio>
+      </ros2_control> -->
       <gazebo>
-        <plugin filename="ign_ros2_control-system" name="ign_ros2_control::IgnitionROS2ControlPlugin">
+        <plugin filename="ign_ros2_control-system"
+                name="ign_ros2_control::IgnitionROS2ControlPlugin">
           <parameters>$(find balltze_bringup)/config/controllers.yaml</parameters>
+        </plugin>
+      </gazebo>
+      <gazebo>
+        <plugin filename="libignition-gazebo-contact-system.so"
+                name="ignition::gazebo::systems::Contact">
+        </plugin>
+      </gazebo>
+      <gazebo>
+        <plugin
+          filename="ignition-gazebo-imu-system"
+          name="ignition::gazebo::systems::Imu">
         </plugin>
       </gazebo>

File: balltze_description/urdf/hardware.ros2_control.xacro (robot description, xacro)
@@ -2,5 +2,5 @@
 <robot xmlns:xacro="http://wiki.ros.org/xacro">
     <xacro:macro name="ros2_control_system">
-      <xacro:macro name="ros2_control_joint" params="joint_name motor_id">
+      <xacro:macro name="ros2_control_joint" params="joint_name motor_id inverted">
         <joint name="${joint_name}">
           <command_interface name="position" />
@@ -11,12 +11,8 @@
           <state_interface name="effort" />
           <param name="id">${motor_id}</param>
+          <param name="inverted">${inverted}</param>
         </joint>
       </xacro:macro>
-      <xacro:macro name="leg_joints" params="leg_prefix coxa_motor_id">
-        <xacro:ros2_control_joint joint_name="${leg_prefix}_body_link_to_coxa_link_joint" motor_id="${coxa_motor_id}"/>
-        <xacro:ros2_control_joint joint_name="${leg_prefix}_coxa_link_to_femur_link_joint" motor_id="${coxa_motor_id+1}"/>
-        <xacro:ros2_control_joint joint_name="${leg_prefix}_femur_link_to_tibia_link_joint" motor_id="${coxa_motor_id+2}"/>
-      </xacro:macro>
-      <ros2_control name="DynamixelSystem" type="system">
+      <ros2_control name="DynamixelSystemf" type="system">
         <hardware>
           <plugin>balltze_dynamixel_system/BalltzeDynamixelSystem</plugin>
@@ -25,8 +21,24 @@
           <param name="return_delay">50</param>
         </hardware>
-        <xacro:leg_joints leg_prefix="front_left"  coxa_motor_id="1" />
-        <xacro:leg_joints leg_prefix="front_right" coxa_motor_id="4" />
-        <xacro:leg_joints leg_prefix="rear_left"   coxa_motor_id="7" />
-        <xacro:leg_joints leg_prefix="rear_right"  coxa_motor_id="10" />
+        <xacro:ros2_control_joint joint_name="fl_joint_1" motor_id="1" inverted="true"  />
+        <xacro:ros2_control_joint joint_name="fl_joint_2" motor_id="2" inverted="true"  />
+        <xacro:ros2_control_joint joint_name="fl_joint_3" motor_id="3" inverted="false" />
+        <xacro:ros2_control_joint joint_name="fr_joint_1" motor_id="4" inverted="true"  />
+        <xacro:ros2_control_joint joint_name="fr_joint_2" motor_id="5" inverted="false" />
+        <xacro:ros2_control_joint joint_name="fr_joint_3" motor_id="6" inverted="true"  />
+      </ros2_control>
+      <ros2_control name="DynamixelSystemr" type="system">
+        <hardware>
+          <plugin>balltze_dynamixel_system/BalltzeDynamixelSystem</plugin>
+          <param name="serial_port">/dev/ttyUSB2</param>
+          <param name="baudrate">1000000</param>
+          <param name="return_delay">50</param>
+        </hardware>
+        <xacro:ros2_control_joint joint_name="rl_joint_1" motor_id="1" inverted="false" />
+        <xacro:ros2_control_joint joint_name="rl_joint_2" motor_id="2" inverted="true"  />
+        <xacro:ros2_control_joint joint_name="rl_joint_3" motor_id="3" inverted="false" />
+        <xacro:ros2_control_joint joint_name="rr_joint_1" motor_id="4" inverted="false" />
+        <xacro:ros2_control_joint joint_name="rr_joint_2" motor_id="5" inverted="false" />
+        <xacro:ros2_control_joint joint_name="rr_joint_3" motor_id="6" inverted="true"  />
       </ros2_control>
     </xacro:macro>
